File: kicad/zzelia65.kicad_pcb (KiCad board)
At the start: 2 copper layers, 0 parts

Commit message: initial pcb
Parts:
- added D_0: D_Small, Diode_THT:D_DO-35_SOD27_P7.62mm_Horizontal, F.Cu at (204.0, 232.6)
- added D_1: D_Small, Diode_THT:D_DO-35_SOD27_P7.62mm_Horizontal, F.Cu at (322.5, 228.4)
- added D_2: D_Small, Diode_THT:D_DO-35_SOD27_P7.62mm_Horizontal, F.Cu at (420.1, 130.3)
- added D_3: D_Small, Diode_THT:D_DO-35_SOD27_P7.62mm_Horizontal, F.Cu at (342.7, 207.5)
- added D_4: D_Small, Diode_THT:D_DO-35_SOD27_P7.62mm_Horizontal, F.Cu at (342.7, 204.0)
- added D_5: D_Small, Diode_THT:D_DO-35_SOD27_P7.62mm_Horizontal, F.Cu at (420.1, 126.7)
- added D_6: D_Small, Diode_THT:D_DO-35_SOD27_P7.62mm_Horizontal, F.Cu at (322.5, 224.8)
- added D_7: D_Small, Diode_THT:D_DO-35_SOD27_P7.62mm_Horizontal, F.Cu at (300.9, 228.4)
- added D_8: D_Small, Diode_THT:D_DO-35_SOD27_P7.62mm_Horizontal, F.Cu at (426.1, 117.2)
- added D_9: D_Small, Diode_THT:D_DO-35_SOD27_P7.62mm_Horizontal, F.Cu at (367.7, 183.8)
- added D_B1: D_Small, Diode_THT:D_DO-35_SOD27_P7.62mm_Horizontal, F.Cu at (426.1, 113.6)
- added D_Back1: D_Small, Diode_THT:D_DO-35_SOD27_P7.62mm_Horizontal, F.Cu at (426.1, 110.1)
- added D_Backslash1: D_Small, Diode_THT:D_DO-35_SOD27_P7.62mm_Horizontal, F.Cu at (426.1, 106.5)
- added D_C1: D_Small, Diode_THT:D_DO-35_SOD27_P7.62mm_Horizontal, F.Cu at (300.9, 231.9)
- added D_Caps1: D_Small, Diode_THT:D_DO-35_SOD27_P7.62mm_Horizontal, F.Cu at (311.7, 228.4)
- added D_Close1: D_Small, Diode_THT:D_DO-35_SOD27_P7.62mm_Horizontal, F.Cu at (311.7, 224.8)
- added D_Comma1: D_Small, Diode_THT:D_DO-35_SOD27_P7.62mm_Horizontal, F.Cu at (311.7, 231.9)
- added D_D1: D_Small, Diode_THT:D_DO-35_SOD27_P7.62mm_Horizontal, F.Cu at (268.6, 228.4)
- added D_Del1: D_Small, Diode_THT:D_DO-35_SOD27_P7.62mm_Horizontal, F.Cu at (300.9, 224.8)
- added D_Dot1: D_Small, Diode_THT:D_DO-35_SOD27_P7.62mm_Horizontal, F.Cu at (290.2, 231.9)
- added D_Down1: D_Small, Diode_THT:D_DO-35_SOD27_P7.62mm_Horizontal, F.Cu at (290.2, 228.4)
- added D_E1: D_Small, Diode_THT:D_DO-35_SOD27_P7.62mm_Horizontal, F.Cu at (290.2, 224.8)
- added D_End1: D_Small, Diode_THT:D_DO-35_SOD27_P7.62mm_Horizontal, F.Cu at (279.4, 231.9)
- added D_Enter1: D_Small, Diode_THT:D_DO-35_SOD27_P7.62mm_Horizontal, F.Cu at (279.4, 228.4)
- added D_Esc1: D_Small, Diode_THT:D_DO-35_SOD27_P7.62mm_Horizontal, F.Cu at (34.9, 28.6)
- added D_F1: D_Small, Diode_THT:D_DO-35_SOD27_P7.62mm_Horizontal, F.Cu at (268.6, 231.9)
- added D_Fn1: D_Small, Diode_THT:D_DO-35_SOD27_P7.62mm_Horizontal, F.Cu at (426.1, 103.0)
- added D_G1: D_Small, Diode_THT:D_DO-35_SOD27_P7.62mm_Horizontal, F.Cu at (268.6, 224.8)
- added D_H1: D_Small, Diode_THT:D_DO-35_SOD27_P7.62mm_Horizontal, F.Cu at (257.8, 231.9)
- added D_Home1: D_Small, Diode_THT:D_DO-35_SOD27_P7.62mm_Horizontal, F.Cu at (257.8, 228.4)
- added D_I1: D_Small, Diode_THT:D_DO-35_SOD27_P7.62mm_Horizontal, F.Cu at (257.8, 224.8)
- added D_Insert1: D_Small, Diode_THT:D_DO-35_SOD27_P7.62mm_Horizontal, F.Cu at (247.1, 231.9)
- added D_J1: D_Small, Diode_THT:D_DO-35_SOD27_P7.62mm_Horizontal, F.Cu at (247.1, 228.4)
- added D_K1: D_Small, Diode_THT:D_DO-35_SOD27_P7.62mm_Horizontal, F.Cu at (279.4, 224.8)
- added D_L1: D_Small, Diode_THT:D_DO-35_SOD27_P7.62mm_Horizontal, F.Cu at (420.1, 123.2)
- added D_LAlt1: D_Small, Diode_THT:D_DO-35_SOD27_P7.62mm_Horizontal, F.Cu at (236.3, 229.0)
- added D_LCtrl1: D_Small, Diode_THT:D_DO-35_SOD27_P7.62mm_Horizontal, F.Cu at (225.5, 232.6)
- added D_LShift1: D_Small, Diode_THT:D_DO-35_SOD27_P7.62mm_Horizontal, F.Cu at (225.5, 225.5)
- added D_LWin1: D_Small, Diode_THT:D_DO-35_SOD27_P7.62mm_Horizontal, F.Cu at (214.8, 232.6)
- added D_Left1: D_Small, Diode_THT:D_DO-35_SOD27_P7.62mm_Horizontal, F.Cu at (225.5, 229.0)
- added D_LetA1: D_Small, Diode_THT:D_DO-35_SOD27_P7.62mm_Horizontal, F.Cu at (236.3, 225.5)
- added D_M1: D_Small, Diode_THT:D_DO-35_SOD27_P7.62mm_Horizontal, F.Cu at (204.0, 225.5)
- added D_Minus1: D_Small, Diode_THT:D_DO-35_SOD27_P7.62mm_Horizontal, F.Cu at (214.8, 229.0)
- added D_N1: D_Small, Diode_THT:D_DO-35_SOD27_P7.62mm_Horizontal, F.Cu at (236.3, 232.6)
- added D_O1: D_Small, Diode_THT:D_DO-35_SOD27_P7.62mm_Horizontal, F.Cu at (204.0, 229.0)
- added D_Open1: D_Small, Diode_THT:D_DO-35_SOD27_P7.62mm_Horizontal, F.Cu at (304.8, 134.5)
- added D_P1: D_Small, Diode_THT:D_DO-35_SOD27_P7.62mm_Horizontal, F.Cu at (304.8, 130.9)
- added D_Plus1: D_Small, Diode_THT:D_DO-35_SOD27_P7.62mm_Horizontal, F.Cu at (304.8, 127.4)
- added D_Q1: D_Small, Diode_THT:D_DO-35_SOD27_P7.62mm_Horizontal, F.Cu at (214.8, 225.5)
- added D_Quote1: D_Small, Diode_THT:D_DO-35_SOD27_P7.62mm_Horizontal, F.Cu at (304.8, 123.8)
- added D_R1: D_Small, Diode_THT:D_DO-35_SOD27_P7.62mm_Horizontal, F.Cu at (182.5, 232.6)
- added D_RAlt1: D_Small, Diode_THT:D_DO-35_SOD27_P7.62mm_Horizontal, F.Cu at (160.9, 229.0)
- added D_RCtrl1: D_Small, Diode_THT:D_DO-35_SOD27_P7.62mm_Horizontal, F.Cu at (193.2, 229.0)
- added D_RShift1: D_Small, Diode_THT:D_DO-35_SOD27_P7.62mm_Horizontal, F.Cu at (193.2, 225.5)
- added D_Right1: D_Small, Diode_THT:D_DO-35_SOD27_P7.62mm_Horizontal, F.Cu at (182.5, 229.0)
- added D_S1: D_Small, Diode_THT:D_DO-35_SOD27_P7.62mm_Horizontal, F.Cu at (182.5, 225.5)
- added D_Semi1: D_Small, Diode_THT:D_DO-35_SOD27_P7.62mm_Horizontal, F.Cu at (171.7, 232.6)
- added D_Slash1: D_Small, Diode_THT:D_DO-35_SOD27_P7.62mm_Horizontal, F.Cu at (160.9, 232.6)
- added D_Space1: D_Small, Diode_THT:D_DO-35_SOD27_P7.62mm_Horizontal, F.Cu at (171.7, 229.0)
- added D_T1: D_Small, Diode_THT:D_DO-35_SOD27_P7.62mm_Horizontal, F.Cu at (171.7, 225.5)
- added D_Tab1: D_Small, Diode_THT:D_DO-35_SOD27_P7.62mm_Horizontal, F.Cu at (193.2, 232.6)
- added D_U1: D_Small, Diode_THT:D_DO-35_SOD27_P7.62mm_Horizontal, F.Cu at (160.9, 225.5)
- added D_Up1: D_Small, Diode_THT:D_DO-35_SOD27_P7.62mm_Horizontal, F.Cu at (229.6, 138.7)
- added D_V1: D_Small, Diode_THT:D_DO-35_SOD27_P7.62mm_Horizontal, F.Cu at (229.6, 135.1)
- added D_W1: D_Small, Diode_THT:D_DO-35_SOD27_P7.62mm_Horizontal, F.Cu at (229.6, 131.6)
- added D_X1: D_Small, Diode_THT:D_DO-35_SOD27_P7.62mm_Horizontal, F.Cu at (229.6, 128.0)
- added D_Y1: D_Small, Diode_THT:D_DO-35_SOD27_P7.62mm_Horizontal, F.Cu at (229.6, 124.5)
- added D_Z1: D_Small, Diode_THT:D_DO-35_SOD27_P7.62mm_Horizontal, F.Cu at (304.8, 138.0)
- added K_0: MX-NoLED, MX:MXOnly-1U-NoLED, F.Cu at (215.9, 25.4)
- added K_1: MX-NoLED, MX:MXOnly-1U-NoLED, F.Cu at (44.5, 25.4)
- added K_2: MX-NoLED, MX:MXOnly-1U-NoLED, F.Cu at (63.5, 25.4)
- added K_3: MX-NoLED, MX:MXOnly-1U-NoLED, F.Cu at (82.5, 25.4)
- added K_4: MX-NoLED, MX:MXOnly-1U-NoLED, F.Cu at (101.6, 25.4)
- added K_5: MX-NoLED, MX:MXOnly-1U-NoLED, F.Cu at (120.7, 25.4)
- added K_6: MX-NoLED, MX:MXOnly-1U-NoLED, F.Cu at (139.7, 25.4)
- added K_7: MX-NoLED, MX:MXOnly-1U-NoLED, F.Cu at (158.8, 25.4)
- added K_8: MX-NoLED, MX:MXOnly-1U-NoLED, F.Cu at (177.8, 25.4)
- added K_9: MX-NoLED, MX:MXOnly-1U-NoLED, F.Cu at (196.8, 25.4)
- added K_A1: MX-NoLED, MX:MXOnly-1U-NoLED, F.Cu at (58.7, 63.5)
- added K_B1: MX-NoLED, MX:MXOnly-1U-NoLED, F.Cu at (144.5, 82.5)
- added K_Back1: MX-NoLED, MX:MXOnly-2U-NoLED, F.Cu at (282.6, 25.4)
- added K_Backslash1: MX-NoLED, MX:MXOnly-1.5U-NoLED, F.Cu at (287.3, 44.5)
- added K_C1: MX-NoLED, MX:MXOnly-1U-NoLED, F.Cu at (106.4, 82.5)
- added K_Caps1: MX-NoLED, MX:MXOnly-1.75U-NoLED, F.Cu at (32.5, 63.5)
- added K_Close1: MX-NoLED, MX:MXOnly-1U-NoLED, F.Cu at (263.5, 44.5)
- added K_Comma1: MX-NoLED, MX:MXOnly-1U-NoLED, F.Cu at (201.6, 82.5)
- added K_D1: MX-NoLED, MX:MXOnly-1U-NoLED, F.Cu at (96.8, 63.5)
- added K_Del1: MX-NoLED, MX:MXOnly-1U-NoLED, F.Cu at (320.7, 82.5)
- added K_Dot1: MX-NoLED, MX:MXOnly-1U-NoLED, F.Cu at (220.7, 82.5)
- added K_Down1: MX-NoLED, MX:MXOnly-1U-NoLED, F.Cu at (296.9, 107.2)
- added K_E1: MX-NoLED, MX:MXOnly-1U-NoLED, F.Cu at (92.1, 44.5)
- added K_End1: MX-NoLED, MX:MXOnly-1U-NoLED, F.Cu at (320.7, 63.5)
- added K_Enter1: MX-NoLED, MX:MXOnly-2.25U-NoLED, F.Cu at (280.2, 63.5)
- added K_Esc1: MX-NoLED, MX:MXOnly-1U-NoLED, F.Cu at (25.4, 25.4)
- added K_F1: MX-NoLED, MX:MXOnly-1U-NoLED, F.Cu at (115.9, 63.5)
- added K_Fn1: MX-NoLED, MX:MXOnly-1U-NoLED, F.Cu at (234.9, 101.6)
- added K_G1: MX-NoLED, MX:MXOnly-1U-NoLED, F.Cu at (134.9, 63.5)
- added K_H1: MX-NoLED, MX:MXOnly-1U-NoLED, F.Cu at (154.0, 63.5)
- added K_Home1: MX-NoLED, MX:MXOnly-1U-NoLED, F.Cu at (320.7, 44.5)
- added K_I1: MX-NoLED, MX:MXOnly-1U-NoLED, F.Cu at (187.3, 44.5)
- added K_Insert1: MX-NoLED, MX:MXOnly-1U-NoLED, F.Cu at (320.7, 25.4)
- added K_J1: MX-NoLED, MX:MXOnly-1U-NoLED, F.Cu at (173.0, 63.5)
- added K_K1: MX-NoLED, MX:MXOnly-1U-NoLED, F.Cu at (192.1, 63.5)
- added K_L1: MX-NoLED, MX:MXOnly-1U-NoLED, F.Cu at (211.1, 63.5)
- added K_LAlt1: MX-NoLED, MX:MXOnly-1.25U-NoLED, F.Cu at (75.4, 101.6)
- added K_LCtrl1: MX-NoLED, MX:MXOnly-1.25U-NoLED, F.Cu at (27.8, 101.6)
- added K_LShift1: MX-NoLED, MX:MXOnly-2.25U-NoLED, F.Cu at (37.3, 82.5)
- added K_LWin1: MX-NoLED, MX:MXOnly-1.25U-NoLED, F.Cu at (51.6, 101.6)
- added K_Left1: MX-NoLED, MX:MXOnly-1U-NoLED, F.Cu at (277.8, 107.2)
- added K_M1: MX-NoLED, MX:MXOnly-1U-NoLED, F.Cu at (182.6, 82.5)
- added K_Minus1: MX-NoLED, MX:MXOnly-1U-NoLED, F.Cu at (234.9, 25.4)
- added K_N1: MX-NoLED, MX:MXOnly-1U-NoLED, F.Cu at (163.5, 82.5)
- added K_O1: MX-NoLED, MX:MXOnly-1U-NoLED, F.Cu at (206.4, 44.5)
- added K_Open1: MX-NoLED, MX:MXOnly-1U-NoLED, F.Cu at (244.5, 44.5)
- added K_P1: MX-NoLED, MX:MXOnly-1U-NoLED, F.Cu at (225.4, 44.5)
- added K_Plus1: MX-NoLED, MX:MXOnly-1U-NoLED, F.Cu at (254.0, 25.4)
- added K_Q1: MX-NoLED, MX:MXOnly-1U-NoLED, F.Cu at (54.0, 44.5)
- added K_Quote1: MX-NoLED, MX:MXOnly-1U-NoLED, F.Cu at (249.2, 63.5)
- added K_R1: MX-NoLED, MX:MXOnly-1U-NoLED, F.Cu at (111.1, 44.5)
- added K_RAlt1: MX-NoLED, MX:MXOnly-1U-NoLED, F.Cu at (215.9, 101.6)
- added K_RCtrl1: MX-NoLED, MX:MXOnly-1U-NoLED, F.Cu at (254.0, 101.6)
- added K_RShift1: MX-NoLED, MX:MXOnly-1.75U-NoLED, F.Cu at (265.9, 82.5)
- added K_Right1: MX-NoLED, MX:MXOnly-1U-NoLED, F.Cu at (315.9, 107.2)
- added K_S1: MX-NoLED, MX:MXOnly-1U-NoLED, F.Cu at (77.8, 63.5)
- added K_Semi1: MX-NoLED, MX:MXOnly-1U-NoLED, F.Cu at (230.2, 63.5)
- added K_Slash1: MX-NoLED, MX:MXOnly-1U-NoLED, F.Cu at (239.7, 82.5)
- added K_Space1: MX-NoLED, MX:MXOnly-6.25U-NoLED, F.Cu at (146.8, 101.6)
- added K_T1: MX-NoLED, MX:MXOnly-1U-NoLED, F.Cu at (130.2, 44.5)
- added K_Tab1: MX-NoLED, MX:MXOnly-1.5U-NoLED, F.Cu at (30.2, 44.5)
- added K_U1: MX-NoLED, MX:MXOnly-1U-NoLED, F.Cu at (168.3, 44.5)
- added K_Up1: MX-NoLED, MX:MXOnly-1U-NoLED, F.Cu at (296.9, 88.1)
- added K_V1: MX-NoLED, MX:MXOnly-1U-NoLED, F.Cu at (125.4, 82.5)
- added K_W1: MX-NoLED, MX:MXOnly-1U-NoLED, F.Cu at (73.0, 44.5)
- added K_X1: MX-NoLED, MX:MXOnly-1U-NoLED, F.Cu at (87.3, 82.5)
- added K_Y1: MX-NoLED, MX:MXOnly-1U-NoLED, F.Cu at (149.2, 44.5)
- added K_Z1: MX-NoLED, MX:MXOnly-1U-NoLED, F.Cu at (68.3, 82.5)
- added ProMicro1: ProMicro, promicro:ProMicro, F.Cu at (212.2, 132.2)

Commit message: diodes
Parts:
- ProMicro1: moved to B.Cu
- moved D_2 361.4 mm to (73.0, 29.4), turned to 90 degrees
- moved D_1 334.2 mm to (54.0, 29.4), turned to 90 degrees
- moved D_Caps1 314.2 mm to (42.1, 67.2), turned to 90 degrees
- moved D_3 307.5 mm to (92.1, 29.4), turned to 90 degrees
- moved D_5 305.8 mm to (130.2, 29.4), turned to 90 degrees
- moved D_4 290.0 mm to (111.1, 29.4), turned to 90 degrees
- moved D_B1 273.5 mm to (154.0, 86.5), turned to 90 degrees
- moved D_6 261.2 mm to (149.2, 29.4), turned to 90 degrees
- moved D_E1 258.2 mm to (101.6, 48.4), turned to 90 degrees
- moved D_8 254.4 mm to (187.3, 29.4), turned to 90 degrees
- moved D_Tab1 239.8 mm to (39.7, 48.4), turned to 90 degrees
- moved D_7 239.2 mm to (168.3, 29.4), turned to 90 degrees
- moved D_C1 235.3 mm to (115.9, 86.5), turned to 90 degrees
- moved D_Q1 232.9 mm to (63.5, 48.4), turned to 90 degrees
- moved D_Z1 232.8 mm to (77.8, 86.5), turned to 90 degrees
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
Commit message: edges & holes
Parts:
- added REF**: MountingHole_2.2mm_M2_Pad, MountingHole:MountingHole_2.2mm_M2_Pad, F.Cu at (80.2, 82.5)
- added REF**: MountingHole_2.2mm_M2_Pad, MountingHole:MountingHole_2.2mm_M2_Pad, F.Cu at (295.3, 82.5)
- added REF**: MountingHole_2.2mm_M2_Pad, MountingHole:MountingHole_2.2mm_M2_Pad, F.Cu at (202.4, 54.0)
- added REF**: MountingHole_2.2mm_M2_Pad, MountingHole:MountingHole_2.2mm_M2_Pad, F.Cu at (202.4, 120.7)
- added REF**: MountingHole_2.2mm_M2_Pad, MountingHole:MountingHole_2.2mm_M2_Pad, F.Cu at (45.2, 131.0)
- added REF**: MountingHole_2.2mm_M2_Pad, MountingHole:MountingHole_2.2mm_M2_Pad, F.Cu at (45.2, 39.7)
- added REF**: MountingHole_2.2mm_M2_Pad, MountingHole:MountingHole_2.2mm_M2_Pad, F.Cu at (365.9, 39.7)
- added REF**: MountingHole_2.2mm_M2_Pad, MountingHole:MountingHole_2.2mm_M2_Pad, F.Cu at (365.9, 131.0)
- moved D_RCtrl1 38.0 mm to (290.5, 111.1)
- moved D_Back1 37.7 mm to (331.8, 48.4)
- moved D_Backslash1 37.7 mm to (331.8, 67.5)
- moved D_Enter1 37.7 mm to (331.8, 86.5)
- moved D_Left1 37.7 mm to (319.9, 130.2)
- moved D_Plus1 37.7 mm to (296.1, 48.4)
- moved K_Backslash1 37.7 mm to (319.9, 63.5)
- moved K_Close1 37.7 mm to (296.1, 63.5)
- moved D_Fn1 37.7 mm to (277.0, 124.6)
- moved D_6 37.7 mm to (181.8, 48.4)
- moved D_8 37.7 mm to (219.9, 48.4)
- moved D_Comma1 37.7 mm to (243.7, 105.6)
- moved D_E1 37.7 mm to (134.1, 67.5)
- moved D_F1 37.7 mm to (158.0, 86.5)
- moved D_H1 37.7 mm to (196.1, 86.5)
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Other:
- board outline added: 330.2 x 100.8 mm

Commit message: pcb zones
Parts:
- added SW_Reset1: SW_Push, Button_Switch_THT:SW_PUSH_6mm, B.Cu at (323.9, 46.8)
- renumbered D_LetA1 to D_A1
Connections:
- ProMicro1 pad 1: Net-(ProMicro1-Pad1) -> Row_0
- ProMicro1 pad 10: Net-(ProMicro1-Pad10) -> Row_7
- ProMicro1 pad 11: Net-(ProMicro1-Pad11) -> Row_8
- ProMicro1 pad 12: Net-(ProMicro1-Pad12) -> Row_9
- ProMicro1 pad 14: Net-(ProMicro1-Pad14) -> Col_6
- ProMicro1 pad 15: Net-(ProMicro1-Pad15) -> Col_5
- ProMicro1 pad 16: Net-(ProMicro1-Pad16) -> Col_4
- ProMicro1 pad 17: Net-(ProMicro1-Pad17) -> Col_3
- ProMicro1 pad 18: Net-(ProMicro1-Pad18) -> Col_2
- ProMicro1 pad 19: Net-(ProMicro1-Pad19) -> Col_1
- ProMicro1 pad 2: Net-(ProMicro1-Pad2) -> Row_1
- ProMicro1 pad 20: Net-(ProMicro1-Pad20) -> Col_0
- ProMicro1 pad 22: Net-(ProMicro1-Pad22) -> RESET
- ProMicro1 pad 23: Net-(ProMicro1-Pad23) -> GND
- ProMicro1 pad 3: Net-(ProMicro1-Pad3) -> GND
- ProMicro1 pad 4: Net-(ProMicro1-Pad4) -> GND
- ProMicro1 pad 5: Net-(ProMicro1-Pad5) -> Row_2
- ProMicro1 pad 6: Net-(ProMicro1-Pad6) -> Row_3
- ProMicro1 pad 7: Net-(ProMicro1-Pad7) -> Row_4
- ProMicro1 pad 8: Net-(ProMicro1-Pad8) -> Row_5
- ProMicro1 pad 9: Net-(ProMicro1-Pad9) -> Row_6
Routing:
- added copper zone on B.Cu, net GND
- added copper zone on F.Cu, net GND

Commit message: routing
Parts:
- moved SW_Reset1 31.5 mm to (335.8, 76.0)
- moved D_RCtrl1 7.94 mm to (282.6, 111.1), turned to 0 degrees
- moved D_Down1 7.62 mm to (325.4, 116.7), turned to 0 degrees
- moved D_Up1 6.35 mm to (338.9, 80.2), turned to 270 degrees
- moved D_Caps1 0.32 mm to (74.6, 86.5)
- moved D_Esc1 0.12 mm to (67.5, 48.4)
Connections:
- D_7 pad 1: Row_9 -> Row_0
- D_Del1 pad 1: Row_5 -> Row_6
- D_End1 pad 1: Row_5 -> Row_7
- D_Home1 pad 1: Row_6 -> Row_8
- D_Insert1 pad 1: Row_7 -> Row_9
- D_J1 pad 1: Row_7 -> Row_2
- D_M1 pad 1: Row_6 -> Row_3
- D_U1 pad 1: Row_8 -> Row_1
- K_0 pad 1: Col_3 -> Col_5
- K_7 pad 1: Col_6 -> Col_7
- K_8 pad 1: Col_5 -> Col_7
- K_9 pad 1: Col_4 -> Col_6
- K_Back1 pad 1: Col_0 -> Col_2
- K_Backslash1 pad 1: Col_0 -> Col_2
- K_Close1 pad 1: Col_1 -> Col_3
- K_Comma1 pad 1: Col_5 -> Col_6
- K_Dot1 pad 1: Col_4 -> Col_5
- K_Down1 pad 1: Col_3 -> Col_2
- K_End1 pad 1: Col_0 -> Col_1
- K_Enter1 pad 1: Col_1 -> Col_2
- K_Home1 pad 1: Col_0 -> Col_1
- K_I1 pad 1: Col_5 -> Col_7
- K_Insert1 pad 1: Col_0 -> Col_1
- K_J1 pad 1: Col_6 -> Col_7
- K_K1 pad 1: Col_5 -> Col_6
- K_L1 pad 1: Col_4 -> Col_5
- K_Left1 pad 1: Col_4 -> Col_3
- K_M1 pad 1: Col_6 -> Col_7
- K_Minus1 pad 1: Col_2 -> Col_4
- K_O1 pad 1: Col_4 -> Col_6
- K_Open1 pad 1: Col_2 -> Col_4
- K_P1 pad 1: Col_3 -> Col_5
- K_Plus1 pad 1: Col_1 -> Col_3
- K_Quote1 pad 1: Col_2 -> Col_3
- K_RCtrl1 pad 1: Col_5 -> Col_4
- K_RShift1 pad 1: Col_2 -> Col_3
- K_Right1 pad 1: Col_2 -> Col_1
- K_Semi1 pad 1: Col_3 -> Col_4
- K_Slash1 pad 1: Col_3 -> Col_4
- K_U1 pad 1: Col_6 -> Col_7
- K_Up1 pad 1: Col_1 -> Col_2
- ProMicro1 pad 13: Net-(ProMicro1-Pad13) -> Col_1
- ProMicro1 pad 14: Col_6 -> Col_2
- ProMicro1 pad 15: Col_5 -> Col_3
- ProMicro1 pad 17: Col_3 -> Col_5
- ProMicro1 pad 18: Col_2 -> Col_6
- ProMicro1 pad 19: Col_1 -> Col_7
Routing:
- net Col_3: track 0.00 -> 477.3 mm
- net Col_2: track 0.00 -> 471.6 mm
- net Col_1: track 0.00 -> 464.1 mm
- net Col_4: track 0.00 -> 406.3 mm
- net Col_0: track 0.00 -> 384.8 mm
- net Col_5: track 0.00 -> 380.9 mm
- net Row_4: track 0.00 -> 379.1 mm
- net Row_3: track 0.00 -> 365.7 mm
- net Row_2: track 0.00 -> 344.9 mm
- net Row_1: track 0.00 -> 333.3 mm
- net Col_6: track 0.00 -> 318.0 mm
- net Row_0: track 0.00 -> 308.5 mm
- net Col_7: track 0.00 -> 283.1 mm
- net Row_5: track 0.00 -> 201.6 mm
- net Row_6: track 0.00 -> 170.0 mm
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
Commit message: remove reset button
Parts:
- removed SW_Reset1: SW_Push, Button_Switch_THT:SW_PUSH_6mm
Routing:
- net RESET: track 37.2 -> 0.00 mm
- net Col_1: track 464.1 -> 465.3 mm
Changed lines of the file:
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@@
     (thickness 1.6)
     (drawings 8)
-    (tracks 594)
+    (tracks 588)
     (zones 0)
-    (modules 146)
+    (modules 145)
     (nets 91)
   )
@@
     (add_net Row_9)
   )
-  (module Button_Switch_THT:SW_PUSH_6mm (layer B.Cu)
-    (at 335.75 76)
-    (descr https://www.omron.com/ecb/products/pdf/en-b3f.pdf)
-    (tags "tact sw push 6mm")
-    (fp_text reference SW_Reset1 (at 3.25 2) (layer B.SilkS)
-      (effects (font (size 1 1) (thickness 0.15)) (justify mirror))
-    )
-    (fp_text value SW_Push (at 3.75 -6.7) (layer B.Fab)
-      (effects (font (size 1 1) (thickness 0.15)) (justify mirror))
-    )
-    (fp_line (start 3.25 0.75) (end 6.25 0.75) (layer B.Fab) (width 0.1))
-    (fp_line (start 6.25 0.75) (end 6.25 -5.25) (layer B.Fab) (width 0.1))
-    (fp_line (start 6.25 -5.25) (end 0.25 -5.25) (layer B.Fab) (width 0.1))
-    (fp_line (start 0.25 -5.25) (end 0.25 0.75) (layer B.Fab) (width 0.1))
-    (fp_line (start 0.25 0.75) (end 3.25 0.75) (layer B.Fab) (width 0.1))
-    (fp_line (start 7.75 -6) (end 8 -6) (layer B.CrtYd) (width 0.05))
-    (fp_line (start 8 -6) (end 8 -5.75) (layer B.CrtYd) (width 0.05))
-    (fp_line (start 7.75 1.5) (end 8 1.5) (layer B.CrtYd) (width 0.05))
-    (fp_line (start 8 1.5) (end 8 1.25) (layer B.CrtYd) (width 0.05))
-    (fp_line (start -1.5 1.25) (end -1.5 1.5) (layer B.CrtYd) (width 0.05))
-    (fp_line (start -1.5 1.5) (end -1.25 1.5) (layer B.CrtYd) (width 0.05))
-    (fp_line (start -1.5 -5.75) (end -1.5 -6) (layer B.CrtYd) (width 0.05))
-    (fp_line (start -1.5 -6) (end -1.25 -6) (layer B.CrtYd) (width 0.05))
-    (fp_line (start -1.25 1.5) (end 7.75 1.5) (layer B.CrtYd) (width 0.05))
-    (fp_line (start -1.5 -5.75) (end -1.5 1.25) (layer B.CrtYd) (width 0.05))
-    (fp_line (start 7.75 -6) (end -1.25 -6) (layer B.CrtYd) (width 0.05))
-    (fp_line (start 8 1.25) (end 8 -5.75) (layer B.CrtYd) (width 0.05))
-    (fp_line (start 1 -5.5) (end 5.5 -5.5) (layer B.SilkS) (width 0.12))
-    (fp_line (start -0.25 -1.5) (end -0.25 -3) (layer B.SilkS) (width 0.12))
-    (fp_line (start 5.5 1) (end 1 1) (layer B.SilkS) (width 0.12))
-    (fp_line (start 6.75 -3) (end 6.75 -1.5) (layer B.SilkS) (width 0.12))
-    (fp_circle (center 3.25 -2.25) (end 1.25 -2.5) (layer B.Fab) (width 0.1))
-    (fp_text user %R (at 3.25 -2.25) (layer B.Fab)
-      (effects (font (size 1 1) (thickness 0.15)) (justify mirror))
-    )
-    (pad 2 thru_hole circle (at 0 -4.5 270) (size 2 2) (drill 1.1) (layers *.Cu *.Mask)
-      (net 89 RESET))
-    (pad 1 thru_hole circle (at 0 0 270) (size 2 2) (drill 1.1) (layers *.Cu *.Mask)
-      (net 88 GND))
-    (pad 2 thru_hole circle (at 6.5 -4.5 270) (size 2 2) (drill 1.1) (layers *.Cu *.Mask)
-      (net 89 RESET))
-    (pad 1 thru_hole circle (at 6.5 0 270) (size 2 2) (drill 1.1) (layers *.Cu *.Mask)
-      (net 88 GND))
-    (model ${KISYS3DMOD}/Button_Switch_THT.3dshapes/SW_PUSH_6mm.wrl
-      (at (xyz 0 0 0))
-      (scale (xyz 1 1 1))
-      (rotate (xyz 0 0 0))
-    )
-  )
   (module MountingHole:MountingHole_2.2mm_M2_Pad (layer F.Cu)
     (at 80.16875 82.55)
@@
   (segment (start 94.526249 103.911251) (end 94.526249 99.939011) (width 0.25) (layer B.Cu) (net 79))
   (segment (start 80.3275 118.11) (end 94.526249 103.911251) (width 0.25) (layer B.Cu) (net 79))
-  (segment (start 344.64625 126.712252) (end 344.64625 123.66625) (width 0.25) (layer B.Cu) (net 79))
-  (segment (start 339.234582 132.12392) (end 344.64625 126.712252) (width 0.25) (layer B.Cu) (net 79))
-  (segment (start 92.179446 132.12392) (end 339.234582 132.12392) (width 0.25) (layer B.Cu) (net 79))
-  (segment (start 80.3275 120.271974) (end 92.179446 132.12392) (width 0.25) (layer B.Cu) (net 79))
-  (segment (start 80.3275 118.11) (end 80.3275 120.271974) (width 0.25) (layer B.Cu) (net 79))
   (segment (start 349.338751 99.129999) (end 349.40875 99.06) (width 0.25) (layer B.Cu) (net 79))
   (segment (start 349.338751 118.973749) (end 349.338751 99.129999) (width 0.25) (layer B.Cu) (net 79))
@@
   (segment (start 350.533749 78.885001) (end 350.533749 62.084999) (width 0.25) (layer B.Cu) (net 79))
   (segment (start 349.40875 80.01) (end 350.533749 78.885001) (width 0.25) (layer B.Cu) (net 79))
-  (segment (start 349.40875 60.96) (end 349.40875 41.91) (width 0.25) (layer B.Cu) (net 79))
-  (segment (start 349.40875 64.006002) (end 349.40875 60.96) (width 0.25) (layer B.Cu) (net 79))
-  (segment (start 347.057252 66.3575) (end 349.40875 64.006002) (width 0.25) (layer B.Cu) (net 79))
-  (segment (start 345.59875 66.3575) (end 347.057252 66.3575) (width 0.25) (layer B.Cu) (net 79))
+  (segment (start 80.3275 120.271974) (end 80.3275 118.11) (width 0.25) (layer B.Cu) (net 79))
+  (segment (start 93.555526 133.5) (end 80.3275 120.271974) (width 0.25) (layer B.Cu) (net 79))
+  (segment (start 337.858502 133.5) (end 93.555526 133.5) (width 0.25) (layer B.Cu) (net 79))
+  (segment (start 344.64625 126.712252) (end 337.858502 133.5) (width 0.25) (layer B.Cu) (net 79))
+  (segment (start 344.64625 123.66625) (end 344.64625 126.712252) (width 0.25) (layer B.Cu) (net 79))
+  (segment (start 346.723751 65.232499) (end 345.59875 66.3575) (width 0.25) (layer B.Cu) (net 79))
+  (segment (start 346.723751 62.054009) (end 346.723751 65.232499) (width 0.25) (layer B.Cu) (net 79))
+  (segment (start 347.81776 60.96) (end 346.723751 62.054009) (width 0.25) (layer B.Cu) (net 79))
+  (segment (start 349.40875 60.96) (end 347.81776 60.96) (width 0.25) (layer B.Cu) (net 79))
+  (segment (start 349.40875 41.91) (end 349.40875 60.96) (width 0.25) (layer B.Cu) (net 79))
   (segment (start 114.654998 99.06) (end 116.04625 99.06) (width 0.25) (layer B.Cu) (net 80))
   (segment (start 104.14 109.574998) (end 114.654998 99.06) (width 0.25) (layer B.Cu) (net 80))
@@
   (segment (start 99.3775 77.47) (end 100.80625 78.89875) (width 0.25) (layer F.Cu) (net 87))
   (segment (start 93.82125 77.47) (end 99.3775 77.47) (width 0.25) (layer F.Cu) (net 87))
-  (segment (start 346.723751 44.622501) (end 345.59875 43.4975) (width 0.25) (layer B.Cu) (net 89))
-  (segment (start 346.723751 64.290999) (end 346.723751 44.622501) (width 0.25) (layer B.Cu) (net 89))
-  (segment (start 346.072249 64.942501) (end 346.723751 64.290999) (width 0.25) (layer B.Cu) (net 89))
-  (segment (start 345.348747 64.942501) (end 346.072249 64.942501) (width 0.25) (layer B.Cu) (net 89))
-  (segment (start 342.25 68.041248) (end 345.348747 64.942501) (width 0.25) (layer B.Cu) (net 89))
-  (segment (start 342.25 71.5) (end 342.25 68.041248) (width 0.25) (layer B.Cu) (net 89))
-  (segment (start 335.75 71.5) (end 342.25 71.5) (width 0.25) (layer B.Cu) (net 89))
   (segment (start 197.00875 53.596974) (end 197.00875 60.96) (width 0.25) (layer B.Cu) (net 90))
   (segment (start 187.48375 44.071974) (end 197.00875 53.596974) (width 0.25) (layer B.Cu) (net 90))
@@
   (segment (start 201.77125 89.535) (end 211.29625 99.06) (width 0.25) (layer B.Cu) (net 90))
   (segment (start 201.77125 80.01) (end 201.77125 89.535) (width 0.25) (layer B.Cu) (net 90))
-  (segment (start 217.183749 62.084999) (end 216.05875 60.96) (width 0.25) (layer B.Cu) (net 90))
-  (segment (start 217.183749 82.256249) (end 217.183749 62.084999) (width 0.25) (layer B.Cu) (net 90))
-  (segment (start 211.29625 88.143748) (end 217.183749 82.256249) (width 0.25) (layer B.Cu) (net 90))
-  (segment (start 211.29625 99.06) (end 211.29625 88.143748) (width 0.25) (layer B.Cu) (net 90))
   (segment (start 206.53375 43.943998) (end 206.53375 41.91) (width 0.25) (layer B.Cu) (net 90))
   (segment (start 216.05875 53.468998) (end 206.53375 43.943998) (width 0.25) (layer B.Cu) (net 90))
@@
   (segment (start 298.735998 35.72502) (end 302.324979 39.314001) (width 0.25) (layer B.Cu) (net 90))
   (segment (start 206.53375 41.91) (end 212.71873 35.72502) (width 0.25) (layer B.Cu) (net 90))
+  (segment (start 211.861251 98.494999) (end 211.29625 99.06) (width 0.25) (layer B.Cu) (net 90))
+  (segment (start 211.861251 63.566509) (end 211.861251 98.494999) (width 0.25) (layer B.Cu) (net 90))
+  (segment (start 214.46776 60.96) (end 211.861251 63.566509) (width 0.25) (layer B.Cu) (net 90))
+  (segment (start 216.05875 60.96) (end 214.46776 60.96) (width 0.25) (layer B.Cu) (net 90))
   (zone (net 88) (net_name GND) (layer F.Cu) (hatch edge 0.508)
     (connect_pads (clearance 0.508))
