File: kicad/zzelia65.kicad_pcb (KiCad board)
At the start: 2 copper layers, 330.2 x 100.8 mm, 145 parts

Commit message: reset button
Parts:
- added Reset1: RESET, Button_Switch_THT:SW_PUSH_6mm, B.Cu at (299.8, 46.8)
Routing:
- net RESET: track 0.00 -> 50.1 mm

Commit message: custom components
Parts:
- D_0, D_1, D_2, D_3, D_4, D_5, D_6, D_7, D_8, D_9, D_A1, D_B1, D_Back1, D_Backslash1, D_C1, D_Caps1, D_Close1, D_Comma1, D_D1, D_Del1, D_Dot1, D_Down1, D_E1, D_End1, D_Enter1, D_Esc1, D_F1, D_Fn1, D_G1, D_H1, D_Home1, D_I1, D_Insert1, D_J1, D_K1, D_L1, D_LAlt1, D_LCtrl1, D_LShift1, D_LWin1, D_Left1, D_M1, D_Minus1, D_N1, D_O1, D_Open1, D_P1, D_Plus1, D_Q1, D_Quote1, D_R1, D_RAlt1, D_RCtrl1, D_RShift1, D_Right1, D_S1, D_Semi1, D_Slash1, D_Space1, D_T1, D_Tab1, D_U1, D_Up1, D_V1, D_W1, D_X1, D_Y1, D_Z1: footprint Diode_THT:D_DO-35_SOD27_P7.62mm_Horizontal -> zzelia65:D_DO-35_SOD27_P7.62mm_Horizontal
- ProMicro1: footprint promicro:ProMicro -> zzelia65:ProMicro
- REF** (x8): footprint MountingHole:MountingHole_2.2mm_M2_Pad -> zzelia65:MountingHole_2.2mm_M2_Pad
Other:
- board text added: "github.com/zzeneg/zzelia65 v0.1"

Commit message: JLCPCB text
Other:
- board text added: "JLCJLCJLCJLC"
Changed lines of the file:
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@@
   (general
     (thickness 1.6)
-    (drawings 9)
+    (drawings 10)
     (tracks 594)
     (zones 0)
@@
   (page A3)
   (layers
-    (0 F.Cu signal)
-    (31 B.Cu signal)
+    (0 F.Cu signal hide)
+    (31 B.Cu signal hide)
     (32 B.Adhes user)
     (33 F.Adhes user)
@@
       (net 1 "Net-(D_0-Pad2)"))
   )
+  (gr_text JLCJLCJLCJLC (at 179.35 36.55) (layer B.SilkS)
+    (effects (font (size 1.5 1.5) (thickness 0.3)))
+  )
   (gr_text "github.com/zzeneg/zzelia65 v0.1" (at 179.35 133.3) (layer F.SilkS)

Commit message: add cover
Parts:
- moved D_Backslash1 0.49 mm to (331.3, 67.5)
- moved D_Enter1 0.49 mm to (331.3, 86.6)
- moved D_Semi1 0.49 mm to (271.8, 86.6)
- moved K_Backslash1 0.49 mm to (319.4, 63.6)
- moved K_Close1 0.49 mm to (295.6, 63.6)
- moved K_Slash1 0.49 mm to (271.8, 101.7)
- moved D_Back1 0.49 mm to (331.3, 48.5)
- moved D_Plus1 0.49 mm to (295.6, 48.5)
- moved D_Left1 0.49 mm to (319.4, 130.2)
- moved D_C1 0.49 mm to (147.9, 105.6)
- moved D_Comma1 0.49 mm to (243.2, 105.6)
- moved D_E1 0.49 mm to (133.7, 67.5)
- moved D_F1 0.49 mm to (157.5, 86.6)
- moved D_H1 0.49 mm to (195.6, 86.6)
- moved D_I1 0.49 mm to (228.9, 67.5)
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Other:
- net class Default removed
